File: PCB_design/Pot_panel_v1.00_print.sch (EAGLE design)
At the start: 5 parts

Commit message: Change arduino layout to fit to the buyable clone
Parts:
- removed CON_POT2: (no value), con-lstb:MA06-1
- added SV1: (no value), con-lstb:MA08-1
- added SV2: (no value), con-lstb:MA04-1
Connections:
- new net IO1: SV1.1, SV2.4
- new net IO2: SV1.2, SV2.3
- net A0: now also SV1.6; no longer CON_POT2.4
- net A1: now also SV1.5; no longer CON_POT2.3
- net A2: now also SV1.4; no longer CON_POT2.2
- net A3: now also SV1.3; no longer CON_POT2.1
- net GND: now also SV1.8, SV2.1; no longer CON_POT2.6
- net VCC: now also SV1.7, SV2.2; no longer CON_POT2.5
Changed lines of the file:
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@@
 <part name="SUPPLY9" library="supply2" deviceset="GND" device=""/>
 <part name="P+12" library="supply1" deviceset="VCC" device=""/>
-<part name="CON_POT2" library="con-lstb" deviceset="MA06-1" device=""/>
 <part name="R1" library="pot" deviceset="TRIM_EU-" device="CA6V"/>
 <part name="R2" library="pot" deviceset="TRIM_EU-" device="CA6V"/>
@@
 <part name="SUPPLY3" library="supply2" deviceset="GND" device=""/>
 <part name="SUPPLY4" library="supply2" deviceset="GND" device=""/>
+<part name="SV1" library="con-lstb" deviceset="MA08-1" device=""/>
+<part name="SV2" library="con-lstb" deviceset="MA04-1" device=""/>
+<part name="P+5" library="supply1" deviceset="VCC" device=""/>
+<part name="SUPPLY5" library="supply2" deviceset="GND" device=""/>
 </parts>
 <sheets>
@@
 <instance part="SUPPLY9" gate="GND" x="73.66" y="124.46"/>
 <instance part="P+12" gate="VCC" x="71.12" y="124.46" rot="R180"/>
-<instance part="CON_POT2" gate="1" x="68.58" y="137.16" rot="R270"/>
 <instance part="R1" gate="1" x="86.36" y="104.14" rot="R90"/>
 <instance part="R2" gate="1" x="71.12" y="104.14" rot="R90"/>
@@
 <instance part="SUPPLY3" gate="GND" x="60.96" y="101.6"/>
 <instance part="SUPPLY4" gate="GND" x="48.26" y="101.6"/>
+<instance part="SV1" gate="1" x="63.5" y="137.16" rot="R270"/>
+<instance part="SV2" gate="1" x="40.64" y="137.16" rot="R270"/>
+<instance part="P+5" gate="VCC" x="38.1" y="127" rot="R180"/>
+<instance part="SUPPLY5" gate="GND" x="35.56" y="127"/>
 </instances>
 <busses>
@@
 <pinref part="SUPPLY9" gate="GND" pin="GND"/>
 <wire x1="73.66" y1="127" x2="73.66" y2="129.54" width="0.1524" layer="91"/>
-<pinref part="CON_POT2" gate="1" pin="6"/>
+<pinref part="SV1" gate="1" pin="8"/>
 </segment>
 <segment>
@@
 <pinref part="SUPPLY4" gate="GND" pin="GND"/>
 </segment>
+<segment>
+<pinref part="SV2" gate="1" pin="1"/>
+<pinref part="SUPPLY5" gate="GND" pin="GND"/>
+</segment>
 </net>
 <net name="A3" class="0">
@@
 <wire x1="43.18" y1="109.22" x2="60.96" y2="121.92" width="0.1524" layer="91"/>
 <wire x1="60.96" y1="121.92" x2="60.96" y2="129.54" width="0.1524" layer="91"/>
-<pinref part="CON_POT2" gate="1" pin="1"/>
 <pinref part="R4" gate="1" pin="S"/>
+<pinref part="SV1" gate="1" pin="3"/>
 </segment>
 </net>
@@
 <wire x1="63.5" y1="129.54" x2="63.5" y2="114.3" width="0.1524" layer="91"/>
 <wire x1="63.5" y1="114.3" x2="55.88" y2="109.22" width="0.1524" layer="91"/>
-<pinref part="CON_POT2" gate="1" pin="2"/>
 <pinref part="R3" gate="1" pin="S"/>
+<pinref part="SV1" gate="1" pin="4"/>
 </segment>
 </net>
@@
 <wire x1="71.12" y1="109.22" x2="66.04" y2="114.3" width="0.1524" layer="91"/>
 <wire x1="66.04" y1="114.3" x2="66.04" y2="129.54" width="0.1524" layer="91"/>
-<pinref part="CON_POT2" gate="1" pin="3"/>
 <pinref part="R2" gate="1" pin="S"/>
+<pinref part="SV1" gate="1" pin="5"/>
 </segment>
 </net>
@@
 <pinref part="P+12" gate="VCC" pin="VCC"/>
 <wire x1="71.12" y1="127" x2="71.12" y2="129.54" width="0.1524" layer="91"/>
-<pinref part="CON_POT2" gate="1" pin="5"/>
+<pinref part="SV1" gate="1" pin="7"/>
 </segment>
 <segment>
@@
 <pinref part="P+4" gate="VCC" pin="VCC"/>
 </segment>
+<segment>
+<pinref part="SV2" gate="1" pin="2"/>
+<pinref part="P+5" gate="VCC" pin="VCC"/>
+</segment>
 </net>
 <net name="A0" class="0">
 <segment>
-<pinref part="CON_POT2" gate="1" pin="4"/>
 <wire x1="86.36" y1="109.22" x2="68.58" y2="121.92" width="0.1524" layer="91"/>
 <wire x1="68.58" y1="121.92" x2="68.58" y2="129.54" width="0.1524" layer="91"/>
 <pinref part="R1" gate="1" pin="S"/>
+<pinref part="SV1" gate="1" pin="6"/>
 </segment>
 </net>
+<net name="IO1" class="0">
+<segment>
+<pinref part="SV1" gate="1" pin="1"/>
+<wire x1="55.88" y1="129.54" x2="55.88" y2="127" width="0.1524" layer="91"/>
+<pinref part="SV2" gate="1" pin="4"/>
+<wire x1="55.88" y1="127" x2="43.18" y2="127" width="0.1524" layer="91"/>
+<wire x1="43.18" y1="127" x2="43.18" y2="129.54" width="0.1524" layer="91"/>
+</segment>
+</net>
+<net name="IO2" class="0">
+<segment>
+<pinref part="SV1" gate="1" pin="2"/>
+<wire x1="58.42" y1="129.54" x2="58.42" y2="124.46" width="0.1524" layer="91"/>
+<pinref part="SV2" gate="1" pin="3"/>
+<wire x1="58.42" y1="124.46" x2="40.64" y2="124.46" width="0.1524" layer="91"/>
+<wire x1="40.64" y1="124.46" x2="40.64" y2="129.54" width="0.1524" layer="91"/>
+</segment>
+</net>
