File: PCB_design/RGB_controller_2zone_v1.00_printable.brd (EAGLE design)
At the start: 75.9 x 64.8 mm, 24 parts, among them Q1 IRF512, Q2 IRF512, Q3 IRF512, Q4 IRF512, Q5 IRF512, Q6 IRF512

Commit message: Change arduino layout to fit to the buyable clone
Parts:
- removed CON_POT2: (no value), con-lstb:MA06-1
- added SV1: (no value), con-lstb:MA08-1
- U$1: value PRO-MINI-2 -> ABK-PRO-MINI; device Arduino-clone:PRO-MINI-2 -> Arduino-clone:ABK-PRO-MINI
- moved U$1 7.41 mm to (54.6, 43.2)
Connections:
- new net D12: SV1.1, U$1.D12
- new net D13: SV1.2, U$1.D13
- net A0: now also SV1.6; no longer CON_POT2.4
- net A1: now also SV1.5; no longer CON_POT2.3
- net A2: now also SV1.4; no longer CON_POT2.2
- net A3: now also SV1.3; no longer CON_POT2.1
- net GND: now also SV1.8; no longer CON_POT2.6
- net VCC: now also SV1.7; no longer CON_POT2.5
Routing:
- net N$1: track 295.9 -> 38.4 mm
- net +12V: track 173.3 -> 241.8 mm
- net N$2: track 72.3 -> 23.4 mm
- net N$5: track 0.00 -> 38.1 mm
- net GND: track 288.1 -> 266.6 mm
- net N$3: track 144.1 -> 161.7 mm
- net D13: track 0.00 -> 7.62 mm
- net D12: track 0.00 -> 7.62 mm
- net GATE_1: track 27.5 -> 21.9 mm
- net IC_PWM_OUT_3: track 6.66 -> 12.0 mm
- net VCC: track 5.08 -> 7.62 mm
- net A3: track 5.08 -> 7.62 mm
- net A2: track 5.08 -> 7.62 mm
- net A1: track 5.08 -> 7.62 mm
- net A0: track 5.08 -> 7.62 mm
Other:
- board text removed: "12V"
- board text removed: "GND"
